File: boards/sensor/sensor.kicad_pcb (KiCad board)
At the start: 2 copper layers, 37 x 46 mm, 8 parts, among them J1 Conn_01x04_Female, J2 Conn_01x04_Female, J3 Conn_01x04_Female, J4 Conn_01x04_Female

Commit message: Submitted board
Parts:
- added REF**: MountingHole_3mm_Pad, MountingHole:MountingHole_3mm_Pad, F.Cu at (38.0, -41.0)
- added REF**: MountingHole_3mm_Pad, MountingHole:MountingHole_3mm_Pad, F.Cu at (16.5, -19.0)
- added REF**: MountingHole_3mm_Pad, MountingHole:MountingHole_3mm_Pad, F.Cu at (17.0, -53.0)
Routing:
- net +5V: track 16.1 -> 12.1 mm
Other:
- outline, holes or cut-outs redrawn
- rule pad_to_mask_clearance: 0.05 -> 0.0508
- rule via_min_drill: 0.3 -> 0.254
- rule via_min_size: 0.4 -> 0.51
- board text added: "5V"
- board text added: "5V GND"
- board text added: "5V GND SDA SCL"
- board text added: "G"
- board text added: "L A 5V GND"
- board text added: "USB"
Changed lines of the file:
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@@
   (general
     (thickness 1.6)
-    (drawings 9)
-    (tracks 81)
+    (drawings 12)
+    (tracks 80)
     (zones 0)
-    (modules 8)
+    (modules 11)
     (nets 30)
   )
@@
     (38 B.Mask user)
     (39 F.Mask user)
-    (40 Dwgs.User user hide)
+    (40 Dwgs.User user)
     (41 Cmts.User user)
     (42 Eco1.User user)
@@
     (47 F.CrtYd user)
     (48 B.Fab user)
-    (49 F.Fab user)
+    (49 F.Fab user hide)
   )
   (setup
@@
     (via_size 0.8)
     (via_drill 0.4)
-    (via_min_size 0.4)
-    (via_min_drill 0.3)
+    (via_min_size 0.51)
+    (via_min_drill 0.254)
     (uvia_size 0.3)
     (uvia_drill 0.1)
@@
     (pad_size 1.524 1.524)
     (pad_drill 0.762)
-    (pad_to_mask_clearance 0.05)
+    (pad_to_mask_clearance 0.0508)
     (aux_axis_origin 0 0)
     (visible_elements FFFFFF7F)
@@
       (outputformat 1)
       (mirror false)
-      (drillshape 1)
+      (drillshape 0)
       (scaleselection 1)
-      (outputdirectory ""))
+      (outputdirectory "gerbers/"))
   )
   (net 0 "")
@@
     (add_net "Net-(A1-Pad9)")
   )
+  (module MountingHole:MountingHole_3mm_Pad (layer F.Cu)
+    (at 38 -41)
+    (descr "Mounting Hole 3mm")
+    (tags "mounting hole 3mm")
+    (attr virtual)
+    (fp_text reference REF** (at 0 -4) (layer F.SilkS) hide
+      (effects (font (size 1 1) (thickness 0.15)))
+    )
+    (fp_text value MountingHole_3mm_Pad (at 0 4) (layer F.Fab)
+      (effects (font (size 1 1) (thickness 0.15)))
+    )
+    (fp_text user %R (at 0.3 0) (layer F.Fab)
+      (effects (font (size 1 1) (thickness 0.15)))
+    )
+    (fp_circle (center 0 0) (end 3 0) (layer Cmts.User) (width 0.15))
+    (fp_circle (center 0 0) (end 3.25 0) (layer F.CrtYd) (width 0.05))
+    (pad 1 thru_hole circle (at 0 0) (size 6 6) (drill 3) (layers *.Cu *.Mask))
+  )
+  (module MountingHole:MountingHole_3mm_Pad (layer F.Cu)
+    (at 16.5 -19)
+    (descr "Mounting Hole 3mm")
+    (tags "mounting hole 3mm")
+    (attr virtual)
+    (fp_text reference REF** (at 0 -4) (layer F.SilkS) hide
+      (effects (font (size 1 1) (thickness 0.15)))
+    )
+    (fp_text value MountingHole_3mm_Pad (at 0 4) (layer F.Fab)
+      (effects (font (size 1 1) (thickness 0.15)))
+    )
+    (fp_text user %R (at 0.3 0) (layer F.Fab)
+      (effects (font (size 1 1) (thickness 0.15)))
+    )
+    (fp_circle (center 0 0) (end 3 0) (layer Cmts.User) (width 0.15))
+    (fp_circle (center 0 0) (end 3.25 0) (layer F.CrtYd) (width 0.05))
+    (pad 1 thru_hole circle (at 0 0) (size 6 6) (drill 3) (layers *.Cu *.Mask))
+  )
+  (module MountingHole:MountingHole_3mm_Pad (layer F.Cu)
+    (at 17 -53)
+    (descr "Mounting Hole 3mm")
+    (tags "mounting hole 3mm")
+    (attr virtual)
+    (fp_text reference REF** (at 0 -4) (layer F.SilkS) hide
+      (effects (font (size 1 1) (thickness 0.15)))
+    )
+    (fp_text value MountingHole_3mm_Pad (at 0 4) (layer F.Fab)
+      (effects (font (size 1 1) (thickness 0.15)))
+    )
+    (fp_text user %R (at 0.3 0) (layer F.Fab)
+      (effects (font (size 1 1) (thickness 0.15)))
+    )
+    (fp_circle (center 0 0) (end 3 0) (layer Cmts.User) (width 0.15))
+    (fp_circle (center 0 0) (end 3.25 0) (layer F.CrtYd) (width 0.05))
+    (pad 1 thru_hole circle (at 0 0) (size 6 6) (drill 3) (layers *.Cu *.Mask))
+  )
   (module Connector_PinHeader_2.54mm:PinHeader_1x04_P2.54mm_Vertical (layer F.Cu)
     (at 30 -52.5 90)
     (descr "Through hole straight pin header, 1x04, 2.54mm pitch, single row")
     (tags "Through hole pin header THT 1x04 2.54mm single row")
-    (fp_text reference i2c2 (at 0 -2.33 90) (layer F.SilkS)
+    (fp_text reference i2c2 (at 0 10 90) (layer F.SilkS) hide
       (effects (font (size 1 1) (thickness 0.15)))
     )
@@
     (descr "Arduino Nano, http://www.mouser.com/pdfdocs/Gravitech_Arduino_Nano3_0.pdf")
     (tags "Arduino Nano")
-    (fp_text reference A1 (at 7.62 -5.08) (layer F.SilkS)
+    (fp_text reference A1 (at 7.62 -5.08) (layer F.SilkS) hide
       (effects (font (size 1 1) (thickness 0.15)))
     )
@@
     (descr "Through hole straight pin header, 1x04, 2.54mm pitch, single row")
     (tags "Through hole pin header THT 1x04 2.54mm single row")
-    (fp_text reference J4 (at 0 -2.33 90) (layer F.SilkS)
+    (fp_text reference J4 (at 0 -2.33 90) (layer F.SilkS) hide
       (effects (font (size 1 1) (thickness 0.15)))
     )
@@
     (descr "Through hole straight pin header, 1x04, 2.54mm pitch, single row")
     (tags "Through hole pin header THT 1x04 2.54mm single row")
-    (fp_text reference J1 (at 0 -2.33 90) (layer F.SilkS)
+    (fp_text reference J1 (at 0 -2.33 90) (layer F.SilkS) hide
       (effects (font (size 1 1) (thickness 0.15)))
     )
@@
     (descr "Through hole straight pin header, 1x04, 2.54mm pitch, single row")
     (tags "Through hole pin header THT 1x04 2.54mm single row")
-    (fp_text reference J3 (at 0 -2.33 90) (layer F.SilkS)
+    (fp_text reference J3 (at 0 -2.33 90) (layer F.SilkS) hide
       (effects (font (size 1 1) (thickness 0.15)))
     )
@@
     (descr "Through hole straight pin header, 1x04, 2.54mm pitch, single row")
     (tags "Through hole pin header THT 1x04 2.54mm single row")
-    (fp_text reference J2 (at 0 -2.33 90) (layer F.SilkS)
+    (fp_text reference J2 (at 0 -2.33 90) (layer F.SilkS) hide
       (effects (font (size 1 1) (thickness 0.15)))
     )
@@
     (descr "Through hole straight pin header, 1x02, 2.54mm pitch, single row")
     (tags "Through hole pin header THT 1x02 2.54mm single row")
-    (fp_text reference Power1 (at 0 -2.33 90) (layer F.SilkS)
+    (fp_text reference Power1 (at 0 -2.33 90) (layer F.SilkS) hide
       (effects (font (size 1 1) (thickness 0.15)))
     )
@@
     (descr "Through hole straight pin header, 1x04, 2.54mm pitch, single row")
     (tags "Through hole pin header THT 1x04 2.54mm single row")
-    (fp_text reference i2c1 (at 0 -2.33 90) (layer F.SilkS)
+    (fp_text reference i2c1 (at 0 10 90) (layer F.SilkS) hide
       (effects (font (size 1 1) (thickness 0.15)))
     )
@@
     )
   )
+  (gr_text G (at 7.5 -45.5) (layer F.SilkS)
+    (effects (font (size 1 1) (thickness 0.15)))
+  )
+  (gr_text 5V (at 27.5 -46) (layer F.SilkS)
+    (effects (font (size 1 1) (thickness 0.15)))
+  )
+  (gr_text "5V GND\n" (at 34 -15.5) (layer F.SilkS)
+    (effects (font (size 1 1) (thickness 0.15)))
+  )
+  (gr_text "5V GND SDA SCL" (at 34 -50) (layer F.SilkS)
+    (effects (font (size 1 1) (thickness 0.15)))
+  )
+  (gr_text "L  A  5V GND" (at 34.5 -36.5) (layer F.SilkS)
+    (effects (font (size 1 1) (thickness 0.15)))
+  )
+  (gr_text USB (at 16.5 -14) (layer F.SilkS)
+    (effects (font (size 1 1) (thickness 0.15)))
+  )
   (gr_poly (pts (xy 42 -13) (xy 5 -13) (xy 5 -59) (xy 42 -59)) (layer Edge.Cuts) (width 0.1))
-  (gr_circle (center 38 -41) (end 41 -41) (layer Edge.Cuts) (width 0.15))
-  (gr_circle (center 16.5 -19) (end 19.5 -19) (layer Edge.Cuts) (width 0.05))
-  (gr_circle (center 17 -53) (end 20 -53) (layer Edge.Cuts) (width 0.05))
   (gr_line (start 16.5 -13) (end 16.5 -19) (layer Eco1.User) (width 0.15))
   (gr_line (start 17 -59) (end 17 -53) (layer Eco1.User) (width 0.15))
@@
   (segment (start 19.294999 -45.794999) (end 19.294999 -46.294999) (width 1) (layer B.Cu) (net 16))
   (segment (start 19.294999 -45.794999) (end 19.294999 -46.794999) (width 1) (layer B.Cu) (net 16))
-  (segment (start 18.92 -46.42) (end 23 -50.5) (width 2) (layer B.Cu) (net 16))
-  (segment (start 28.5 -18) (end 32.5 -18) (width 2) (layer F.Cu) (net 26))
+  (segment (start 18.42 -45.92) (end 22.5 -50) (width 2) (layer B.Cu) (net 16))
   (segment (start 27.5 -46) (end 30 -48.5) (width 2) (layer F.Cu) (net 26))
   (segment (start 27.5 -38.5) (end 28.5 -37.5) (width 2) (layer B.Cu) (net 26))
